File: A1-FlightComputer-Hardware/A1-FlightComputer.kicad_pcb (KiCad board)
At the start: 4 copper layers, 73.6 x 73.6 mm, 101 parts, among them J201 Conn_01x01_Socket, J202 Conn_01x01_Socket, J203 Conn_01x02_Socket, J204 Conn_01x02_Socket, J205 Conn_02x05_Odd_Even, J301 Conn_01x07_Socket, J302 Conn_01x03_Socket, J303 Conn_01x04_Socket, J304 Conn_01x02_Socket, J305 Conn_01x02_Socket, J306 Conn_01x02_Socket, J401 PWR_IN, J402 USB_B_Micro, Q301 PMOS, SW201 SW_Push, SW202 SW_Push, SW203 SW_SPDT, SW301 SW_SPST, SW401 SW_SPST, U201 STM32L475RCTx, U202 W25N01GVZEIG, U301 BMP390, U302 LSM6DSOTR, U303 DRV8212P, U304 ADXL314, U401 AZ1117-5.0, U402 AZ1117-3.3, Y201 32.768kHz LSE, Y202 8MHz HSE

Commit message: Flight computer V2
Parts:
- removed C305: 0.1uF 5V, Capacitor_SMD:C_0603_1608Metric_Pad1.08x0.95mm_HandSolder
- removed C306: 0.1uF 6V, Capacitor_SMD:C_0603_1608Metric_Pad1.08x0.95mm_HandSolder
- removed J201, J202: Conn_01x01_Socket, Connector_PinSocket_2.54mm:PinSocket_1x01_P2.54mm_Vertical
- removed the J301 at (154.4, 111.0)
- removed the J302 at (168.6, 106.0)
- removed J303: Conn_01x04_Socket, Connector_PinSocket_2.54mm:PinSocket_1x04_P2.54mm_Vertical
- removed J306: Conn_01x02_Socket, Connector_PinSocket_2.54mm:PinSocket_1x02_P2.54mm_Vertical
- removed the JP201 at (136.6, 65.1)
- removed the JP202 at (136.6, 67.7)
- removed JP301: SolderJumper_2_Bridged, Jumper:SolderJumper-2_P1.3mm_Bridged_RoundedPad1.0x1.5mm
- removed the R303 at (165.5, 104.6)
- removed SW301: SW_SPST, Connector_PinHeader_2.54mm:PinHeader_1x02_P2.54mm_Vertical
- removed the TP202 at (163.4, 103.4)
- removed the U303 at (185.3, 65.3)
- Q301: value PMOS -> Q_NMOS_GSD; footprint Package_TO_SOT_SMD:SOT-143 -> Package_TO_SOT_SMD:SOT-23
- moved TP207 21.8 mm to (139.6, 91.8)
- moved R306 17.9 mm to (133.7, 112.0), turned to -90 degrees
- moved R305 14.7 mm to (137.7, 112.0), turned to -90 degrees
- moved SW203 14.6 mm to (129.3, 63.5), turned to -90 degrees
- moved R303 14.1 mm to (145.7, 112.0), turned to -90 degrees
- moved D304 13.6 mm to (133.7, 107.0), turned to -90 degrees
- moved R304 13.2 mm to (141.7, 112.0), turned to -90 degrees
- moved J204 12.9 mm to (152.7, 111.0), turned to 90 degrees
- moved TP204 11.7 mm to (137.2, 47.8)
- moved D303 8.90 mm to (137.7, 107.0), turned to -90 degrees
- moved R207 8.36 mm to (151.5, 63.2), turned to -90 degrees
- moved TP403 8.32 mm to (137.1, 54.9)
- moved D301 7.84 mm to (145.7, 107.0), turned to -90 degrees
- moved D302 6.20 mm to (141.7, 107.0), turned to -90 degrees
- moved TP203 6.01 mm to (169.8, 103.7)
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- renumbered D404 to D402, D402 to D403, D403 to D404, J304 to J301, J305 to J302, JP203 to JP201, JP204 to JP202, R304 to R303, R305 to R304, R306 to R305, R307 to R306, TP203 to TP202, TP204 to TP203, TP205 to TP204, TP206 to TP205, TP207 to TP206, TP208 to TP207, TP209 to TP208, U304 to U303
Connections:
- D402 pad 1: +5V -> +BATT
- J301 pad 2: Net-(J304-Pin_2) -> Net-(J301-Pin_2)
- Q301 pad 1: Net-(J304-Pin_2) -> /Peripherals/Buzzer_ON
- Q301 pad 2: /Peripherals/GoPro_ON -> GND
- Q301 pad 3: GND -> Net-(J301-Pin_2)
- TP203 pad 1: /Peripherals/GoPro_ON -> /Peripherals/Buzzer_ON
- U201 pad 14: /Peripherals/STG3 -> unconnected-(U201-PA0-Pad14)
- U201 pad 15: /Peripherals/STG2 -> unconnected-(U201-PA1-Pad15)
- U201 pad 16: /Peripherals/STG1 -> unconnected-(U201-PA2-Pad16)
- U201 pad 17: /Peripherals/STG0 -> unconnected-(U201-PA3-Pad17)
- U201 pad 28: /Peripherals/Payload_TEMP -> unconnected-(U201-PB2-Pad28)
- U201 pad 33: /Peripherals/GoPro_ON -> /Peripherals/Buzzer_ON
- U201 pad 36: /STM32/PB15 -> unconnected-(U201-PB15-Pad36)
- U201 pad 53: /STM32/PC12 -> unconnected-(U201-PC12-Pad53)
- U201 pad 58: Net-(JP201-A) -> unconnected-(U201-PB6-Pad58)
- U201 pad 59: Net-(JP202-A) -> unconnected-(U201-PB7-Pad59)
- U201 pad 61: /Peripherals/Actuator_IN1 -> unconnected-(U201-PB8-Pad61)
- U201 pad 62: /Peripherals/Actuator_IN2 -> unconnected-(U201-PB9-Pad62)
- U303 pad 25: (no net) -> unconnected-(U303-NC-Pad25)
Routing:
- net /Peripherals/Actuator_IN1: track 41.1 -> 0.00 mm, vias 2 -> 0
- net /Peripherals/Actuator_IN2: track 40.3 -> 0.00 mm, vias 2 -> 0
- net /STM32/PB15: track 40.2 -> 0.00 mm, vias 1 -> 0
- net /Peripherals/GoPro_ON: track 33.5 -> 0.00 mm, vias 1 -> 0
- net /Peripherals/STG3: track 30.6 -> 0.00 mm
- net /Peripherals/Payload_TEMP: track 29.5 -> 0.00 mm, vias 1 -> 0
- net /Peripherals/STG2: track 28.8 -> 0.00 mm
- net /Peripherals/Buzzer_ON: track 0.00 -> 28.7 mm
- net Net-(JP201-A): track 27.2 -> 0.00 mm
- net /Peripherals/STG1: track 26.7 -> 0.00 mm
- net Net-(JP202-A): track 25.5 -> 0.00 mm
- net /Peripherals/STG0: track 25.0 -> 0.00 mm
- net /STM32/PC12: track 19.5 -> 0.00 mm, vias 1 -> 0
- net /Peripherals/LED0: track 20.7 -> 34.6 mm
- net /Peripherals/LoRa_TX: track 10.9 -> 0.00 mm
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- added copper zone on F.Cu, net Net-(J301-Pin_2)
- removed copper zone on F.Cu, net Net-(J303-Pin_4)
- removed copper zone on F.Cu, net Net-(J304-Pin_2)
- removed copper zone on F.Cu, net Net-(JP301-B)
Other:
- board size 73.6 x 73.6 mm -> 74.8 x 74.8 mm
- board text added: "3V3 CONN"
- board text added: "5V CONN"
- board text added: "BUZZER"
- board text added: "Buzzer"
- board text added: "Flight Computer Version 2.0"
- board text added: "JTAG CONN"
- board text added: "PB8"
- board text added: "PB9"
- board text removed: "+SW"
- board text removed: "Actuator"
- board text removed: "CAM_ON"
- board text removed: "Camera"
- board text removed: "Flight Computer Version 1.0"
- board text removed: "LoRa Switch"
- board text removed: "LoRa Transmitter"
- board text removed: "OUT1"
- board text removed: "OUT2"
- board text removed: "PB15"
- board text removed: "PC12"
- board text removed: "STG0"
- board text removed: "STG1"
- board text removed: "STG2"
- board text removed: "STG3"
- board text removed: "Strain Gauges"
- board text removed: "TEMP"
- board text removed: "Temperature"
