File: A1-FlightComputer-Hardware/A1-FlightComputer.kicad_sch (KiCad schematic)
At the start: 4 parts

Commit message: Flight computer V2
Other:
- sheet Peripherals ports: added Buzzer_ON; removed Actuator_IN1, Actuator_IN2, GoPro_ON, LoRa_RX, LoRa_TX, Payload_TEMP, STG0, STG1, STG2, STG3
- sheet STM32 ports: added Buzzer_ON; removed Actuator_IN1, Actuator_IN2, GoPro_ON, LoRa_RX, LoRa_TX, Payload_TEMP, STG0, STG1, STG2, STG3
- note removed: "USB Debug USB OTG ST-Link Programming Pressure / Temperature / Humidity Low Accelleration IMU High Accelleration IMU I/O Breakout ADC Battery Checking 2x UART 1x I2C 4x GPIO Strain Guages 1x GPIO (A) Payload Temp 2x GPIO LEDs SPI Flash Chip SDMMC SD card? Payload temp sensors Payload linear actuator"
