File: A1-FlightComputer-Hardware/peripherals.kicad_sch (KiCad schematic)
At the start: 30 parts, among them J301 Conn_01x07_Socket, J302 Conn_01x03_Socket, J303 Conn_01x04_Socket, J304 Conn_01x02_Socket, J305 Conn_01x02_Socket, J306 Conn_01x02_Socket, Q301 PMOS, SW301 SW_SPST, U301 BMP390, U302 LSM6DSOTR, U303 DRV8212P, U304 ADXL314

Commit message: Flight computer V2
Parts:
- removed C305, C306: 100nF, Capacitor_SMD:C_0603_1608Metric_Pad1.08x0.95mm_HandSolder, symbol Device:C
- removed J301: Conn_01x07_Socket, Connector_PinSocket_2.54mm:PinSocket_1x07_P2.54mm_Vertical, symbol Connector:Conn_01x07_Socket
- removed J302: Conn_01x03_Socket, Connector_PinSocket_2.54mm:PinSocket_1x03_P2.54mm_Vertical, symbol Connector:Conn_01x03_Socket
- removed J303: Conn_01x04_Socket, Connector_PinSocket_2.54mm:PinSocket_1x04_P2.54mm_Vertical, symbol Connector:Conn_01x04_Socket
- removed J306: Conn_01x02_Socket, Connector_PinSocket_2.54mm:PinSocket_1x02_P2.54mm_Vertical, symbol Connector:Conn_01x02_Socket
- removed JP301: SolderJumper_2_Bridged, Jumper:SolderJumper-2_P1.3mm_Bridged_RoundedPad1.0x1.5mm, symbol Jumper:SolderJumper_2_Bridged
- removed Q301: PMOS, Package_TO_SOT_SMD:SOT-143, symbol Simulation_SPICE:PMOS
- removed R303: 4k7, Resistor_SMD:R_0603_1608Metric_Pad0.98x0.95mm_HandSolder, symbol Device:R
- removed SW301: SW_SPST, Connector_PinHeader_2.54mm:PinHeader_1x02_P2.54mm_Vertical, symbol Switch:SW_SPST
- removed U303: DRV8212P, Package_SON:WSON-8-1EP_2x2mm_P0.5mm_EP0.9x1.6mm_ThermalVias, symbol Driver_Motor:DRV8212P
- added Q301: Q_NMOS_GSD, Package_TO_SOT_SMD:SOT-23, symbol Device:Q_NMOS_GSD
- renumbered J304 to J301, J305 to J302, R304 to R303, R305 to R304, R306 to R305, R307 to R306, U304 to U303
Connections:
- net GND: now also Q301.2 (S)
- net at J301.2 (Pin_2): now also Q301.3 (D)
- new net Buzzer_ON: Q301.1 (G)
Other:
- note added: "Buzzer"
- note removed: "GOPro Power"
- note removed: "LoRa Connection"
- note removed: "Payload DS18B20"
- note removed: "Payload Linear Actuator L12-50-50-6-s"
- note removed: "Strain Guages"
- moved on the sheet: D301, D302, D303, D304, J301, R303, R304, R305, R306
