File: A1-FlightComputer-Hardware/power.kicad_sch (KiCad schematic)
At the start: 19 parts, among them J401 PWR_IN, J402 USB_B_Micro, SW401 SW_SPST, U401 AZ1117-5.0, U402 AZ1117-3.3

Commit message: Flight computer V2
Parts:
- renumbered D404 to D402, D402 to D403, D403 to D404
Connections:
- net +5V: no longer D402.1 (K)
- net +BATT: now also D402.1 (K)
Other:
- note removed: "USB will not be used to power PCB, only for data transport"
- moved on the sheet: D402, J402
